File: Hardware/OSAVC/OSAVC.sch (KiCad schematic (older format))
At the start: 39 parts, among them J1 DIGITAL, J11 I2C1, J12 GPS, J13 Radio, J14 RC RX, J2 COMMUNICATION, J20 Left Motor, J21 Right Motor, J22 Steering, J23 Encoder 4, J28 I2C LiDAR, J3 PWM/DIGITAL, J4 ANALOG 1, J5 POWER, J6 PWM, J7 ANALOG 2, J9 , SW1 BTN, U1 24LC256, U2 Sparkfun_ICM-20948_breakout

Commit message: New hardware schematic complete, bug fix for rc_rx, increase baud rate of uart1
Parts:
- removed C1: 0.1uF, Capacitor_SMD:C_0805_2012Metric, symbol Device:C_Small
- removed C2: 680uF, Capacitor_Tantalum_SMD:CP_EIA-7343-30_AVX-N, symbol Device:CP1
- removed D1, D2, D3, D4, D5: LED, LED_SMD:LED_0805_2012Metric, symbol Device:LED
- removed H1, H2, H3: MountingHole, MountingHole:MountingHole_3mm, symbol Mechanical:MountingHole
- removed J1: DIGITAL, Connector_PinHeader_2.54mm:PinHeader_2x18_P2.54mm_Vertical, symbol Connector_Generic:Conn_02x18_Odd_Even
- removed J11: I2C1, Connector_PinHeader_2.54mm:PinHeader_1x04_P2.54mm_Vertical, symbol Connector_Generic:Conn_01x04
- removed J12: GPS, Connector_PinHeader_2.54mm:PinHeader_1x06_P2.54mm_Vertical, symbol Connector_Generic:Conn_01x06
- removed J13: Radio, Connector_PinHeader_2.54mm:PinHeader_1x06_P2.54mm_Vertical, symbol Connector_Generic:Conn_01x06
- removed J14: RC RX, Connector_PinHeader_2.54mm:PinHeader_1x06_P2.54mm_Vertical, symbol Connector_Generic:Conn_01x06
- removed J2: COMMUNICATION, Connector_PinHeader_2.54mm:PinHeader_1x08_P2.54mm_Vertical, symbol Connector_Generic:Conn_01x08
- removed J20: Left Motor, Connector_PinHeader_2.54mm:PinHeader_1x06_P2.54mm_Vertical, symbol Connector_Generic:Conn_01x06
- removed J21: Right Motor, Connector_PinHeader_2.54mm:PinHeader_1x06_P2.54mm_Vertical, symbol Connector_Generic:Conn_01x06
- removed J22: Steering, Connector_PinHeader_2.54mm:PinHeader_1x06_P2.54mm_Vertical, symbol Connector_Generic:Conn_01x06
- removed J23: Encoder 4, Connector_PinHeader_2.54mm:PinHeader_1x06_P2.54mm_Vertical, symbol Connector_Generic:Conn_01x06
- removed J28: I2C LiDAR, Connector_PinHeader_2.54mm:PinHeader_1x06_P2.54mm_Vertical, symbol Connector_Generic:Conn_01x06
- removed J3: PWM/DIGITAL, Connector_PinHeader_2.54mm:PinHeader_2x08_P2.54mm_Vertical, symbol Connector_Generic:Conn_02x08_Odd_Even
- removed J4: ANALOG 1, Connector_PinHeader_2.54mm:PinHeader_1x08_P2.54mm_Vertical, symbol Connector_Generic:Conn_01x08
- removed J5: POWER, Connector_PinHeader_2.54mm:PinHeader_1x06_P2.54mm_Vertical, symbol Connector_Generic:Conn_01x06
- removed J6: PWM, OSAVC interface shield:PWM_HDR, symbol OSAVC_generated:PWM
- removed J7: ANALOG 2, Connector_PinHeader_2.54mm:PinHeader_1x08_P2.54mm_Vertical, symbol Connector_Generic:Conn_01x08
- removed J9: (no value), Connector_PinHeader_2.54mm:PinHeader_2x08_P2.54mm_Vertical, symbol Connector_Generic:Conn_02x08_Odd_Even
- removed R1: 180K, Resistor_SMD:R_0805_2012Metric, symbol Device:R_US
- removed R2: 11K, Resistor_SMD:R_0805_2012Metric, symbol Device:R_US
- removed R3, R4, R6, R7: 240, Resistor_SMD:R_0805_2012Metric, symbol Device:R_US
- removed R5: 560, Resistor_SMD:R_0805_2012Metric, symbol Device:R_US
- removed R8, R9: 4.7K, Resistor_SMD:R_0805_2012Metric, symbol Device:R_US
- removed SW1: BTN, Button_Switch_THT:SW_PUSH_6mm_H4.3mm, symbol Switch:SW_Push
- removed U1: 24LC256, Package_SO:SOIJ-8_5.3x5.3mm_P1.27mm, symbol Memory_EEPROM:24LC256
- removed U2: Sparkfun_ICM-20948_breakout, OSAVC interface shield:SPARKFUN_ICM20948_BREAKOUT, symbol OSAVC_generated:Sparkfun_ICM-20948_breakout
Connections:
- net labels removed: +3.3V, +3V3, +5V, +BATT, 0, 77, 78, 85, A0, A1, A10, A11, A12, A13, A14, A15, A2, A3, A4, A5, A6, A7, A8, A9, AGND, GND, OC2, OC3, OC4, OC5, RA0, RA1, RA4, RA5, RE0, RE1, RE2, RE3, RE4, RE9, RESET, SCK1, SCK2, SCL1, SCL2, SDA1, SDA2, SDI1, SDI2, SDO1, SDO2, U2RX, U2TX, U4RX, U4TX, U5RX, U5TX
- wire segments 191 -> 0
- no-connect marks 70 -> 0
Other:
- note added: "1.0"
- note added: "OSAVC"
- note added: "September 7 2021"
- note removed: "1.2"
- note removed: "EEPROM"
- note removed: "EXPANSION PWM"
- note removed: "EXT 5V/PWM"
- note removed: "FrSky RX"
- note removed: "GPS M8N"
- note removed: "Headers"
- note removed: "I2C User"
- note removed: "IMU Breakout SPI1"
- note removed: "LiDAR"
- note removed: "March 4, 2021"
- note removed: "OSAVC Interface Board"
- note removed: "Radio Telemetry"
- note removed: "SPI2 Rotary Encoders"
- note removed: "UART Communications"
- note removed: "USE EXT 5V"
