File: Hardware/OSAVC/Microprocessor.sch (KiCad schematic (older format))
At the start: 36 parts, among them J2 ICSP, J3 USB_B_Micro, SW1 SW_Push_Dual, U6 PIC32MX795F512L-80x-PF, U7 FT232RL, Y1 WE 830059082

Commit message: rev 1.1 OSAVC completed
Parts:
- removed SW1: SW_Push_Dual, Button_Switch_THT:SW_PUSH_6mm_H4.3mm, symbol Switch:SW_Push_Dual
- added SW1: SW_Push, Button_Switch_THT:SW_PUSH_6mm_H4.3mm, symbol Switch:SW_Push
- C18: footprint Capacitor_SMD:C_0805_2012Metric_Pad1.18x1.45mm_HandSolder -> Capacitor_SMD:C_0603_1608Metric_Pad1.08x0.95mm_HandSolder
- R10, R11, R9: value 50 -> 51
Connections:
- net GND: now also SW1.1
- net at U6.26 (PGEC2/RB6): now also R10.2; no longer R9.2
- net at U6.27 (PGED2/RB7): now also R9.2; no longer R10.2
- net at R12.2: now also SW1.2
Changed lines of the file:
@@
 F 0 "C18" H 3815 1346 50  0000 L CNN
 F 1 "10uF" H 3815 1255 50  0000 L CNN
-F 2 "Capacitor_SMD:C_0805_2012Metric_Pad1.18x1.45mm_HandSolder" H 3738 1150 50  0001 C CNN
+F 2 "Capacitor_SMD:C_0603_1608Metric_Pad1.08x0.95mm_HandSolder" H 3738 1150 50  0001 C CNN
 F 3 "~" H 3700 1300 50  0001 C CNN
 	1    3700 1300
@@
 	850  1550 850  950
 $Comp
-L Switch:SW_Push_Dual SW1
-U 1 1 6145BCDB
-P 5700 2300
-F 0 "SW1" H 5700 2585 50  0000 C CNN
-F 1 "SW_Push_Dual" H 5700 2494 50  0000 C CNN
-F 2 "Button_Switch_THT:SW_PUSH_6mm_H4.3mm" H 5700 2500 50  0001 C CNN
-F 3 "~" H 5700 2500 50  0001 C CNN
-	1    5700 2300
-	1    0    0    -1
-$EndComp
-$Comp
 L Device:R_US R8
 U 1 1 61460099
@@
 P 6100 2050
 F 0 "R11" V 6000 2050 50  0000 C CNN
-F 1 "50" V 6200 2050 50  0000 C CNN
+F 1 "51" V 6200 2050 50  0000 C CNN
 F 2 "Resistor_SMD:R_0603_1608Metric" V 6140 2040 50  0001 C CNN
 F 3 "~" H 6100 2050 50  0001 C CNN
@@
 P 8350 1850
 F 0 "R9" V 8250 1800 50  0000 C CNN
-F 1 "50" V 8250 1950 50  0000 C CNN
+F 1 "51" V 8250 1950 50  0000 C CNN
 F 2 "Resistor_SMD:R_0603_1608Metric" V 8390 1840 50  0001 C CNN
 F 3 "~" H 8350 1850 50  0001 C CNN
@@
 P 8350 1950
 F 0 "R10" V 8450 1900 50  0000 C CNN
-F 1 "50" V 8450 2050 50  0000 C CNN
+F 1 "51" V 8450 2050 50  0000 C CNN
 F 2 "Resistor_SMD:R_0603_1608Metric" V 8390 1940 50  0001 C CNN
 F 3 "~" H 8350 1950 50  0001 C CNN
@@
 Wire Wire Line
 	4400 2250 4350 2250
-Wire Wire Line
-	7000 2850 4350 2850
 Text GLabel 1850 3050 0    50   Input ~ 0
 SDA1
@@
 	5300 1400 5300 1550
 Wire Wire Line
-	5500 2300 5500 2500
-Wire Wire Line
 	5500 2500 5300 2500
-Connection ~ 5500 2500
 Connection ~ 5300 2500
 Wire Wire Line
-	5900 2300 5900 2500
-Wire Wire Line
 	5900 2500 6300 2500
 Wire Wire Line
 	6300 2500 6300 2450
-Connection ~ 5900 2500
 Wire Wire Line
 	5300 1550 6300 1550
@@
 	8200 1850 7000 1850
 Wire Wire Line
-	7000 1850 7000 2850
-Wire Wire Line
-	7200 2950 7200 1950
-Wire Wire Line
 	7200 1950 8200 1950
-Wire Wire Line
-	4350 2950 7200 2950
 Wire Notes Line
 	7600 1200 9900 1200
@@
 Wire Wire Line
 	1050 3750 1050 3850
+$Comp
+L Switch:SW_Push SW1
+U 1 1 6188781E
+P 5700 2500
+F 0 "SW1" H 5700 2785 50  0000 C CNN
+F 1 "SW_Push" H 5700 2694 50  0000 C CNN
+F 2 "Button_Switch_THT:SW_PUSH_6mm_H4.3mm" H 5700 2700 50  0001 C CNN
+F 3 "~" H 5700 2700 50  0001 C CNN
+	1    5700 2500
+	1    0    0    -1
+$EndComp
+Wire Wire Line
+	7200 1950 7200 2850
+Wire Wire Line
+	4350 2850 7200 2850
+Wire Wire Line
+	7000 1850 7000 2950
+Wire Wire Line
+	7000 2950 4350 2950
 $EndSCHEMATC
