File: Hardware/OSAVC/OSAVC_pwr.sch (KiCad schematic (older format))
At the start: 26 parts, among them J1 Barrel_Jack_Switch, Q1 FDN340P, U1 PTN78060W_EUW-7, U2 LP38690DTX-5.0_NOPB, U3 LP38690DT-3.3_NOPB, U4 MCP6001-OT, U5 PTN78060W_EUW-7

Commit message: rev 1.1 OSAVC completed
Parts:
- removed C7: 2.2uF, Capacitor_SMD:C_0603_1608Metric_Pad1.08x0.95mm_HandSolder, symbol Device:C
- removed C8: 100uF, Capacitor_SMD:C_1210_3225Metric_Pad1.33x2.70mm_HandSolder, symbol Device:CP1
- removed J1: Barrel_Jack_Switch, Connector_BarrelJack:BarrelJack_Wuerth_6941xx301002, symbol Connector:Barrel_Jack_Switch
- removed R6: 21.0K, Resistor_SMD:R_0603_1608Metric, symbol Device:R_US
- removed U1, U5: PTN78060W_EUW-7, Module:Texas_EUW_R-PDSS-T7_THT, symbol Converter_DCDC:PTN78060W_EUW-7
- removed U4: MCP6001-OT, Package_TO_SOT_SMD:SOT-23-5, symbol Amplifier_Operational:MCP6001-OT
- added C7: 0.1uF, Capacitor_SMD:C_0603_1608Metric_Pad1.08x0.95mm_HandSolder, symbol Device:C_Small
- added C8: 10uF, Capacitor_SMD:C_0603_1608Metric_Pad1.08x0.95mm_HandSolder, symbol Device:C
- added J1: Battery In, OSAVC:XT60, symbol Connector:Conn_01x02_Female
- added U1: PTN78020W_EUK-7, Module:Texas_EUK_R-PDSS-T7_THT, symbol Converter_DCDC:PTN78020W_EUK-7
- added U4: MCP6001U, Package_TO_SOT_SMD:SOT-23-5, symbol Amplifier_Operational:MCP6001U
- added U5: MIC29300-5.0WU, MIC293000:MIC29300-5.0WU, symbol MIC293000:MIC29300-5.0WU
- C1: footprint Capacitor_SMD:C_0603_1608Metric_Pad1.08x0.95mm_HandSolder -> Capacitor_SMD:C_0805_2012Metric
- C2: value 100uF -> 330uF; footprint Capacitor_SMD:C_1210_3225Metric_Pad1.33x2.70mm_HandSolder -> OSAVC:EEE-FNA331XUL
- C3, C5: footprint Capacitor_SMD:C_1206_3216Metric_Pad1.33x1.80mm_HandSolder -> Capacitor_SMD:C_0603_1608Metric_Pad1.08x0.95mm_HandSolder
- C4, C6: footprint Capacitor_SMD:C_0805_2012Metric_Pad1.18x1.45mm_HandSolder -> Capacitor_SMD:C_0603_1608Metric_Pad1.08x0.95mm_HandSolder
- Q1: value FDN340P -> AO3423
Connections:
- net +3V3: now also U4.3 (-)
- net +5V: now also U4.5 (V+)
- net +5VA: now also C8.1, U5.3 (OUT)
- net +7V: now also C7.1, U1.6 (VO), U5.1 (IN)
- net +BATT: now also J1.1 (Pin_1), U1.2 (VI)
- net GND: now also C7.2, C8.2, J1.2 (Pin_2), U1.1 (GND), U1.7 (GND), U4.2 (V-), U5.2 (GND), U5.4
- net at R1.1: now also U1.4 (VO_Adj)
- net at R3.2, R5.1: now also U4.1 (+)
- net at Q1.1 (G): now also U4.4
- no-connect marks 4 -> 2
